File: 00-air-temp-monitor.kicad_pcb (KiCad board)
At the start: 2 copper layers, 38.6 x 37.6 mm, 32 parts, among them J1 Conn_01x04, SW1 SW_Push, U1 STM32L011F4Px, U2 TPS62A01APDDC, U3 HS96L03W2C03, U4 AHT20, Y1 32.768kHz

Commit message: Layout update
Parts:
- moved C14 3.50 mm to (121.9, 79.0), turned to 90 degrees
- moved R8 2.47 mm to (113.3, 90.6)
- moved R5 2.34 mm to (102.4, 101.1), turned to -90 degrees
- moved C10 1.54 mm to (99.8, 103.6)
- moved C11 1.54 mm to (99.8, 104.6)
- moved C9 1.54 mm to (99.8, 102.6)
- moved C7 1.19 mm to (94.5, 79.4)
- moved C3 1.02 mm to (103.1, 95.0)
- moved C4 1.02 mm to (103.1, 96.0)
- moved R7 0.89 mm to (115.3, 93.6)
- moved R1 0.84 mm to (95.1, 81.3), turned to 180 degrees
- moved J1 0.65 mm to (110.1, 108.6)
- moved R9 0.30 mm to (120.8, 79.0)
- moved C13 0.26 mm to (101.2, 86.1)
Routing:
- net /I2C1_SCL: track 0.00 -> 38.0 mm, vias 0 -> 1
- net /I2C1_SDA: track 0.00 -> 32.7 mm, vias 0 -> 2
- net +3V3: track 0.00 -> 27.2 mm, vias 0 -> 11
- net /NRST: track 0.00 -> 26.1 mm, vias 0 -> 1
- net +BATT: track 0.00 -> 25.3 mm, vias 0 -> 2
- net /SWCLK: track 0.00 -> 20.0 mm
- net /SWDIO: track 0.00 -> 18.0 mm
- net GND: track 0.00 -> 9.67 mm, vias 0 -> 30
- net Net-(U2-FB): track 0.00 -> 3.65 mm
- net Net-(U2-SW): track 0.00 -> 2.71 mm
- net Net-(L1-Pad2): track 0.00 -> 2.65 mm
- net Net-(U2-PG): track 0.00 -> 1.95 mm
- net Net-(U4-VDD): track 0.00 -> 1.46 mm
- added copper zone on In1.Cu, net +3V3
- added copper zone on F.Cu, net GND
- added copper zone on In2.Cu, net GND
Other:
- outline, holes or cut-outs redrawn
- copper layers 2 -> 4

Commit message: Layout done
Parts:
- R5: footprint Resistor_SMD:R_0805_2012Metric_Pad1.20x1.40mm_HandSolder -> Resistor_SMD:R_0402_1005Metric_Pad0.72x0.64mm_HandSolder
- moved Y1 3.30 mm to (102.9, 92.8)
- moved C5 1.59 mm to (101.2, 91.7), turned to -90 degrees
- moved C6 1.49 mm to (101.2, 94.0), turned to 90 degrees
- moved C12 1.00 mm to (96.0, 101.1)
- moved C10 1.00 mm to (100.8, 103.6)
- moved C11 1.00 mm to (100.8, 104.6)
- moved C8 1.00 mm to (96.5, 108.2)
- moved C9 1.00 mm to (100.8, 102.6)
- moved L1 1.00 mm to (99.5, 100.1)
- moved R2 1.00 mm to (96.5, 107.2)
- moved R3 1.00 mm to (96.5, 106.2)
- moved R4 1.00 mm to (96.5, 106.2)
- moved R6 1.00 mm to (94.0, 103.1)
- moved U2 1.00 mm to (97.0, 103.6)
- moved C3 0.51 mm to (103.1, 95.5)
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Routing:
- net GND: track 9.67 -> 23.0 mm, vias 30 -> 137
- net Net-(U1-PC14): track 0.00 -> 4.78 mm
- net Net-(U1-PC15): track 0.00 -> 4.61 mm
- net Net-(U2-FB): track 3.65 -> 5.50 mm, vias 0 -> 1
- net +3V3: track 27.2 -> 28.9 mm
- net +BATT: track 25.3 -> 26.3 mm
- net Net-(L1-Pad2): track 2.65 -> 1.72 mm
- net /SWDIO: vias 0 -> 1
- net /SWCLK: vias 0 -> 1
- added copper zone on In2.Cu, net +3V3
- added copper zone on B.Cu, net GND
- added copper zone on In1.Cu, net GND
- removed copper zone on In1.Cu, net +3V3
- removed copper zone on In2.Cu, net GND
Other:
- outline, holes or cut-outs redrawn
- board text added: "3V3"
- board text added: "GND"
- board text added: "SWCLK"
- board text added: "SWDIO"

Commit message: Mounting holes added
Parts:
- added H1: MountingHole, MountingHole:MountingHole_2.7mm_M2.5, F.Cu at (87.9, 110.0)
- added H2: MountingHole, MountingHole:MountingHole_2.7mm_M2.5, F.Cu at (119.4, 110.0)
Routing:
- net GND: vias 137 -> 128
