File: 00-air-temp-monitor.kicad_sch (KiCad schematic)
At the start: 31 parts, among them J1 Conn_01x04, SW1 SW_Push, U1 STM32L011F4Px, U2 TPS62A01APDDC, U3 ER_OLEDM0.91_1x-I2C, U4 AHT20, Y1 Crystal

Commit message: Updated schematic
Parts:
- added R9: 330, symbol Device:R
- C14: value 100nF -> 10uF; JLCPCB C2857965 -> C408132
Connections:
- net +3V3: now also R9.2; no longer U4.2 (VDD)
- new net: R9.1, U4.2 (VDD)

Commit message: Updated crystal
Parts:
- BT1: footprint (none) -> thr_Connector:BS-24-B4AK023
- C1, C10, C11, C12, C13, C14, C2, C3, C4, C7, C8, C9: footprint (none) -> Capacitor_SMD:C_0402_1005Metric_Pad0.74x0.62mm_HandSolder
- C5, C6: value 15pF -> 1.5pF; footprint (none) -> Capacitor_SMD:C_0402_1005Metric_Pad0.74x0.62mm_HandSolder; JLCPCB C1548 -> C285112
- J1: footprint (none) -> Connector_PinHeader_2.54mm:PinHeader_1x04_P2.54mm_Vertical
- L1: footprint (none) -> Inductor_SMD:L_1008_2520Metric_Pad1.43x2.20mm_HandSolder
- R1, R2, R3, R4, R6, R7, R8, R9: footprint (none) -> Resistor_SMD:R_0402_1005Metric_Pad0.72x0.64mm_HandSolder
- R5: footprint (none) -> Resistor_SMD:R_0805_2012Metric_Pad1.20x1.40mm_HandSolder
- SW1: footprint (none) -> thr_Switches:Tactile_switch_4.5x4.5x5.0; JLCPCB C51978191 -> C39832245
- U3: value ER_OLEDM0.91_1x-I2C -> HS96L03W2C03; footprint Display:ER_OLEDM0.91_1x-I2C -> thr_Display:HS96L03W2C03
- U4: footprint (none) -> thr_Temperature:AHT20; MPN (none) -> AHT20
- Y1: value Crystal -> 32.768kHz; footprint (none) -> Crystal:Crystal_SMD_2012-2Pin_2.0x1.2mm_HandSoldering; JLCPCB C3034396 -> C276418
Changed lines of the file:
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@@
 			)
 		)
-		(property "Footprint" ""
+		(property "Footprint" "Capacitor_SMD:C_0402_1005Metric_Pad0.74x0.62mm_HandSolder"
 			(at 154.6352 39.37 0)
 			(hide yes)
@@
 			)
 		)
-		(property "Footprint" ""
+		(property "Footprint" "Capacitor_SMD:C_0402_1005Metric_Pad0.74x0.62mm_HandSolder"
 			(at 64.4652 41.91 0)
 			(hide yes)
@@
 			)
 		)
-		(property "Footprint" ""
+		(property "Footprint" "Capacitor_SMD:C_0402_1005Metric_Pad0.74x0.62mm_HandSolder"
 			(at 174.9552 85.09 0)
 			(hide yes)
@@
 			)
 		)
-		(property "Footprint" ""
+		(property "Footprint" "thr_Switches:Tactile_switch_4.5x4.5x5.0"
 			(at 74.93 102.87 0)
 			(hide yes)
@@
 			)
 		)
-		(property "JLCPCB" "C51978191"
+		(property "JLCPCB" "C39832245"
 			(at 80.01 102.87 90)
 			(hide yes)
@@
 			)
 		)
-		(property "Footprint" ""
+		(property "Footprint" "Capacitor_SMD:C_0402_1005Metric_Pad0.74x0.62mm_HandSolder"
 			(at 166.0652 39.37 0)
 			(hide yes)
@@
 			)
 		)
-		(property "Value" "15pF"
+		(property "Value" "1.5pF"
 			(at 135.89 125.7299 0)
 			(show_name no)
@@
 			)
 		)
-		(property "Footprint" ""
+		(property "Footprint" "Capacitor_SMD:C_0402_1005Metric_Pad0.74x0.62mm_HandSolder"
 			(at 133.0452 128.27 0)
 			(hide yes)
@@
 			)
 		)
-		(property "JLCPCB" "C1548"
+		(property "JLCPCB" "C285112"
 			(at 132.08 124.46 0)
 			(hide yes)
@@
 			)
 		)
-		(property "Footprint" ""
+		(property "Footprint" "thr_Connector:BS-24-B4AK023"
 			(at 39.37 37.846 90)
 			(hide yes)
@@
 			)
 		)
-		(property "Value" "15pF"
+		(property "Value" "1.5pF"
 			(at 110.49 125.7299 0)
 			(show_name no)
@@
 			)
 		)
-		(property "Footprint" ""
+		(property "Footprint" "Capacitor_SMD:C_0402_1005Metric_Pad0.74x0.62mm_HandSolder"
 			(at 107.6452 128.27 0)
 			(hide yes)
@@
 			)
 		)
-		(property "JLCPCB" "C1548"
+		(property "JLCPCB" "C285112"
 			(at 106.68 124.46 0)
 			(hide yes)
@@
 			)
 		)
-		(property "Footprint" ""
+		(property "Footprint" "Resistor_SMD:R_0402_1005Metric_Pad0.72x0.64mm_HandSolder"
 			(at 116.332 49.53 90)
 			(hide yes)
@@
 			)
 		)
-		(property "Footprint" ""
+		(property "Footprint" "Resistor_SMD:R_0402_1005Metric_Pad0.72x0.64mm_HandSolder"
 			(at 89.662 21.59 90)
 			(hide yes)
@@
 			)
 		)
-		(property "Footprint" ""
+		(property "Footprint" "Capacitor_SMD:C_0402_1005Metric_Pad0.74x0.62mm_HandSolder"
 			(at 143.2052 39.37 0)
 			(hide yes)
@@
 			)
 		)
-		(property "Footprint" ""
+		(property "Footprint" "Capacitor_SMD:C_0402_1005Metric_Pad0.74x0.62mm_HandSolder"
 			(at 186.3852 85.09 0)
 			(hide yes)
@@
 			)
 		)
-		(property "Footprint" ""
+		(property "Footprint" "Inductor_SMD:L_1008_2520Metric_Pad1.43x2.20mm_HandSolder"
 			(at 101.6 30.48 0)
 			(hide yes)
@@
 			)
 		)
-		(property "Footprint" ""
+		(property "Footprint" "Resistor_SMD:R_0402_1005Metric_Pad0.72x0.64mm_HandSolder"
 			(at 261.62 67.818 90)
 			(hide yes)
@@
 			)
 		)
-		(property "Value" "ER_OLEDM0.91_1x-I2C"
+		(property "Value" "HS96L03W2C03"
 			(at 248.92 44.4499 0)
 			(show_name no)
@@
 			)
 		)
-		(property "Footprint" "Display:ER_OLEDM0.91_1x-I2C"
+		(property "Footprint" "thr_Display:HS96L03W2C03"
 			(at 258.064 55.88 0)
 			(hide yes)
@@
 			)
 		)
-		(property "Footprint" ""
+		(property "Footprint" "Capacitor_SMD:C_0402_1005Metric_Pad0.74x0.62mm_HandSolder"
 			(at 94.9452 106.68 0)
 			(hide yes)
@@
 			)
 		)
-		(property "Footprint" ""
+		(property "Footprint" "Resistor_SMD:R_0402_1005Metric_Pad0.72x0.64mm_HandSolder"
 			(at 116.332 36.83 90)
 			(hide yes)
@@
 			)
 		)
-		(property "Footprint" ""
+		(property "Footprint" "Resistor_SMD:R_0402_1005Metric_Pad0.72x0.64mm_HandSolder"
 			(at 202.692 104.14 90)
 			(hide yes)
@@
 			)
 		)
-		(property "Footprint" ""
+		(property "Footprint" "Resistor_SMD:R_0402_1005Metric_Pad0.72x0.64mm_HandSolder"
 			(at 193.802 104.14 90)
 			(hide yes)
@@
 			)
 		)
-		(property "Footprint" ""
+		(property "Footprint" "Connector_PinHeader_2.54mm:PinHeader_1x04_P2.54mm_Vertical"
 			(at 241.3 120.65 0)
 			(hide yes)
@@
 			)
 		)
-		(property "Footprint" ""
+		(property "Footprint" "Capacitor_SMD:C_0402_1005Metric_Pad0.74x0.62mm_HandSolder"
 			(at 129.2352 40.64 0)
 			(hide yes)
@@
 			)
 		)
-		(property "Footprint" ""
+		(property "Footprint" "thr_Temperature:AHT20"
 			(at 254 85.09 0)
 			(hide yes)
@@
 			)
 		)
+		(property "MPN" "AHT20"
+			(at 254 85.09 0)
+			(hide yes)
+			(show_name no)
+			(do_not_autoplace no)
+			(effects
+				(font
+					(size 1.27 1.27)
+				)
+			)
+		)
 		(pin "6"
 		)
@@
 			)
 		)
-		(property "Footprint" ""
+		(property "Footprint" "Resistor_SMD:R_0805_2012Metric_Pad1.20x1.40mm_HandSolder"
 			(at 110.49 32.258 90)
 			(hide yes)
@@
 			)
 		)
-		(property "Footprint" ""
+		(property "Footprint" "Capacitor_SMD:C_0402_1005Metric_Pad0.74x0.62mm_HandSolder"
 			(at 129.2352 85.09 0)
 			(hide yes)
@@
 			)
 		)
-		(property "Footprint" ""
+		(property "Footprint" "Capacitor_SMD:C_0402_1005Metric_Pad0.74x0.62mm_HandSolder"
 			(at 254.9652 33.02 0)
 			(hide yes)
@@
 			)
 		)
-		(property "Footprint" ""
+		(property "Footprint" "Capacitor_SMD:C_0402_1005Metric_Pad0.74x0.62mm_HandSolder"
 			(at 143.2052 85.09 0)
 			(hide yes)
@@
 			)
 		)
-		(property "Footprint" ""
+		(property "Footprint" "Resistor_SMD:R_0402_1005Metric_Pad0.72x0.64mm_HandSolder"
 			(at 125.222 49.53 90)
 			(hide yes)
@@
 			)
 		)
-		(property "Footprint" ""
+		(property "Footprint" "Capacitor_SMD:C_0402_1005Metric_Pad0.74x0.62mm_HandSolder"
 			(at 268.9352 74.93 0)
 			(hide yes)
@@
 			)
 		)
-		(property "Value" "Crystal"
+		(property "Value" "32.768kHz"
 			(at 119.38 111.76 0)
 			(show_name no)
@@
 			)
 		)
-		(property "Footprint" ""
+		(property "Footprint" "Crystal:Crystal_SMD_2012-2Pin_2.0x1.2mm_HandSoldering"
 			(at 119.38 116.84 0)
 			(hide yes)
@@
 			)
 		)
-		(property "JLCPCB" "C3034396"
+		(property "JLCPCB" "C276418"
 			(at 119.38 116.84 0)
 			(hide yes)
@@
 			)
 		)
-		(property "Footprint" ""
+		(property "Footprint" "Resistor_SMD:R_0402_1005Metric_Pad0.72x0.64mm_HandSolder"
 			(at 78.232 86.36 90)
 			(hide yes)

Commit message: Layout done
Parts:
- BT1: JLCPCB C2902329 -> (none); LCSC Part # (none) -> C2902329
- C1, C11, C13, C3: JLCPCB C2857965 -> (none); LCSC Part # (none) -> C2857965
- C10, C14, C2, C9: JLCPCB C408132 -> (none); LCSC Part # (none) -> C408132
- C12: JLCPCB C20624278 -> (none); LCSC Part # (none) -> C20624278
- C4: JLCPCB C14445 -> (none); LCSC Part # (none) -> C14445
- C5, C6: JLCPCB C285112 -> (none); LCSC Part # (none) -> C285112
- C7, C8: JLCPCB C1548 -> (none); LCSC Part # (none) -> C1548
- J1: JLCPCB C5383113 -> (none); LCSC Part # (none) -> C5383113
- L1: JLCPCB C435392 -> (none); LCSC Part # (none) -> C435392
- R1, R3: JLCPCB C22356213 -> (none); LCSC Part # (none) -> C22356213
- R2: JLCPCB C852792 -> (none); LCSC Part # (none) -> C852792
- R5: footprint Resistor_SMD:R_0805_2012Metric_Pad1.20x1.40mm_HandSolder -> Resistor_SMD:R_0402_1005Metric_Pad0.72x0.64mm_HandSolder; JLCPCB C17477 -> (none); LCSC Part # (none) -> C17168
- R6: JLCPCB C324794 -> (none); LCSC Part # (none) -> C324794
- R7, R8: JLCPCB C25900 -> (none); LCSC Part # (none) -> C25900
- R9: JLCPCB C12246 -> (none); LCSC Part # (none) -> C12246
- SW1: JLCPCB C39832245 -> (none); LCSC Part # (none) -> C39832245
- U1: JLCPCB C87903 -> (none); LCSC Part # (none) -> C87903
- U2: JLCPCB C41730179 -> (none); LCSC Part # (none) -> C41730179
- U3: JLCPCB C5248080 -> (none); LCSC Part # (none) -> C5248080
- U4: JLCPCB C2757850 -> (none); LCSC Part # (none) -> C2757850
- Y1: JLCPCB C276418 -> (none); LCSC Part # (none) -> C276418

Commit message: Mounting holes added
Parts:
- added H1, H2: MountingHole, MountingHole:MountingHole_2.7mm_M2.5, symbol Mechanical:MountingHole
Changed lines of the file:
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@@
 		(at 170.18 113.03)
 	)
+	(bus_entry
+		(at 210.82 104.14)
+		(size 2.54 2.54)
+		(stroke
+			(width 0)
+			(type default)
+		)
+	)
 	(wire
 		(pts
@@
 	)
 	(symbol
+		(lib_id "Mechanical:MountingHole")
+		(at 21.59 184.15 0)
+		(unit 1)
+		(body_style 1)
+		(exclude_from_sim no)
+		(in_bom no)
+		(on_board yes)
+		(in_pos_files yes)
+		(dnp no)
+		(fields_autoplaced yes)
+		(property "Reference" "H1"
+			(at 24.13 182.8799 0)
+			(show_name no)
+			(do_not_autoplace no)
+			(effects
+				(font
+					(size 1.27 1.27)
+				)
+				(justify left)
+			)
+		)
+		(property "Value" "MountingHole"
+			(at 24.13 185.4199 0)
+			(show_name no)
+			(do_not_autoplace no)
+			(effects
+				(font
+					(size 1.27 1.27)
+				)
+				(justify left)
+			)
+		)
+		(property "Footprint" "MountingHole:MountingHole_2.7mm_M2.5"
+			(at 21.59 184.15 0)
+			(hide yes)
+			(show_name no)
+			(do_not_autoplace no)
+			(effects
+				(font
+					(size 1.27 1.27)
+				)
+			)
+		)
+		(property "Datasheet" ""
+			(at 21.59 184.15 0)
+			(hide yes)
+			(show_name no)
+			(do_not_autoplace no)
+			(effects
+				(font
+					(size 1.27 1.27)
+				)
+			)
+		)
+		(property "Description" "Mounting Hole without connection"
+			(at 21.59 184.15 0)
+			(hide yes)
+			(show_name no)
+			(do_not_autoplace no)
+			(effects
+				(font
+					(size 1.27 1.27)
+				)
+			)
+		)
+		(instances
+			(project "00-air-temp-monitor"
+				(path "/77a0b3b4-fa45-47c7-9e72-52985e1769a2"
+					(reference "H1")
+					(unit 1)
+				)
+			)
+		)
+	)
+	(symbol
 		(lib_id "Device:C")
 		(at 153.67 35.56 0)
@@
 					(unit 1)
 				)
+			)
+		)
+	)
+	(symbol
+		(lib_id "Mechanical:MountingHole")
+		(at 41.91 184.15 0)
+		(unit 1)
+		(body_style 1)
+		(exclude_from_sim no)
+		(in_bom no)
+		(on_board yes)
+		(in_pos_files yes)
+		(dnp no)
+		(fields_autoplaced yes)
+		(property "Reference" "H2"
+			(at 44.45 182.8799 0)
+			(show_name no)
+			(do_not_autoplace no)
+			(effects
+				(font
+					(size 1.27 1.27)
+				)
+				(justify left)
+			)
+		)
+		(property "Value" "MountingHole"
+			(at 44.45 185.4199 0)
+			(show_name no)
+			(do_not_autoplace no)
+			(effects
+				(font
+					(size 1.27 1.27)
+				)
+				(justify left)
+			)
+		)
+		(property "Footprint" "MountingHole:MountingHole_2.7mm_M2.5"
+			(at 41.91 184.15 0)
+			(hide yes)
+			(show_name no)
+			(do_not_autoplace no)
+			(effects
+				(font
+					(size 1.27 1.27)
+				)
+			)
+		)
+		(property "Datasheet" ""
+			(at 41.91 184.15 0)
+			(hide yes)
+			(show_name no)
+			(do_not_autoplace no)
+			(effects
+				(font
+					(size 1.27 1.27)
+				)
+			)
+		)
+		(property "Description" "Mounting Hole without connection"
+			(at 41.91 184.15 0)
+			(hide yes)
+			(show_name no)
+			(do_not_autoplace no)
+			(effects
+				(font
+					(size 1.27 1.27)
+				)
+			)
+		)
+		(instances
+			(project "00-air-temp-monitor"
+				(path "/77a0b3b4-fa45-47c7-9e72-52985e1769a2"
+					(reference "H2")
+					(unit 1)
+				)
